File: hardware/bottom plate/invaders.sch (EAGLE design)
At the start: 171 parts, among them U1 32U4, U2 MCP73831, U3 PAM2401, Y1 16MHz

Commit message: Aggressor Firmware Update
Parts:
- added J10: AVR_SPI_PROG_3X2PTH, SparkFun-Connectors:AVR_SPI_PROG_3X2PTH
Connections:
- removed net N$229: R1.1, U1.!RESET
- new net !RST: J10.5, R1.1, U1.!RESET
- net GND: now also J10.6
- net LEFT: now also J10.1
- net R1CK: now also J10.3
- net R1DA: now also J10.4
- net VCC: now also J10.2
Changed lines of the file:
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@@
 <part name="BT1" library="SparkFun-Batteries" deviceset="BATTERY" device="-18650"/>
 <part name="GND155" library="SparkFun-PowerSymbols" deviceset="GND" device=""/>
+<part name="J10" library="SparkFun-Connectors" deviceset="AVR_SPI_PROG_3X2" device="PTH"/>
+<part name="GND146" library="SparkFun-PowerSymbols" deviceset="GND" device=""/>
+<part name="SUPPLY21" library="SparkFun-PowerSymbols" deviceset="VCC" device=""/>
 </parts>
 <sheets>
@@
 <attribute name="VALUE" x="675.64" y="185.166" size="1.778" layer="96" align="top-center"/>
 </instance>
+<instance part="J10" gate="G$1" x="617.22" y="71.12" smashed="yes">
+<attribute name="NAME" x="612.14" y="76.708" size="1.778" layer="95" font="vector"/>
+<attribute name="VALUE" x="612.14" y="63.754" size="1.778" layer="96" font="vector"/>
+</instance>
+<instance part="GND146" gate="1" x="629.92" y="63.5" smashed="yes">
+<attribute name="VALUE" x="629.92" y="63.246" size="1.778" layer="96" align="top-center"/>
+</instance>
+<instance part="SUPPLY21" gate="G$1" x="629.92" y="76.2" smashed="yes">
+<attribute name="VALUE" x="629.92" y="78.994" size="1.778" layer="96" align="bottom-center"/>
+</instance>
 </instances>
 <busses>
@@
 <label x="586.74" y="142.24" size="1.27" layer="95" xref="yes"/>
 </segment>
+<segment>
+<pinref part="J10" gate="G$1" pin="3"/>
+<wire x1="609.6" y1="71.12" x2="607.06" y2="71.12" width="0.1524" layer="91"/>
+<label x="607.06" y="71.12" size="1.27" layer="95" rot="R180" xref="yes"/>
+</segment>
 </net>
 <net name="R1DA" class="0">
@@
 <label x="586.74" y="139.7" size="1.27" layer="95" xref="yes"/>
 </segment>
+<segment>
+<pinref part="J10" gate="G$1" pin="4"/>
+<wire x1="627.38" y1="71.12" x2="629.92" y2="71.12" width="0.1524" layer="91"/>
+<label x="629.92" y="71.12" size="1.27" layer="95" xref="yes"/>
+</segment>
 </net>
 <net name="N$3" class="0">
@@
 <pinref part="C7" gate="G$1" pin="1"/>
 </segment>
+<segment>
+<pinref part="J10" gate="G$1" pin="2"/>
+<wire x1="627.38" y1="73.66" x2="629.92" y2="73.66" width="0.1524" layer="91"/>
+<wire x1="629.92" y1="73.66" x2="629.92" y2="76.2" width="0.1524" layer="91"/>
+<pinref part="SUPPLY21" gate="G$1" pin="VCC"/>
+</segment>
 </net>
 <net name="GND" class="0">
@@
 <pinref part="GND155" gate="1" pin="GND"/>
 </segment>
+<segment>
+<pinref part="J10" gate="G$1" pin="6"/>
+<wire x1="627.38" y1="68.58" x2="629.92" y2="68.58" width="0.1524" layer="91"/>
+<wire x1="629.92" y1="68.58" x2="629.92" y2="66.04" width="0.1524" layer="91"/>
+<pinref part="GND146" gate="1" pin="GND"/>
+</segment>
 </net>
 <net name="N$1" class="0">
@@
 </segment>
 </net>
-<net name="N$229" class="0">
+<net name="!RST" class="0">
 <segment>
 <pinref part="U1" gate="U1" pin="!RESET"/>
@@
 <wire x1="546.1" y1="203.2" x2="546.1" y2="205.74" width="0.1524" layer="91"/>
 <pinref part="R1" gate="G$1" pin="1"/>
+<wire x1="546.1" y1="203.2" x2="538.48" y2="203.2" width="0.1524" layer="91"/>
+<junction x="546.1" y="203.2"/>
+<label x="538.48" y="203.2" size="1.27" layer="95" rot="R180" xref="yes"/>
+</segment>
+<segment>
+<pinref part="J10" gate="G$1" pin="5"/>
+<wire x1="609.6" y1="68.58" x2="607.06" y2="68.58" width="0.1524" layer="91"/>
+<label x="607.06" y="68.58" size="1.27" layer="95" rot="R180" xref="yes"/>
 </segment>
 </net>
@@
 <label x="586.74" y="137.16" size="1.27" layer="95" xref="yes"/>
 </segment>
+<segment>
+<pinref part="J10" gate="G$1" pin="1"/>
+<wire x1="609.6" y1="73.66" x2="607.06" y2="73.66" width="0.1524" layer="91"/>
+<label x="607.06" y="73.66" size="1.27" layer="95" rot="R180" xref="yes"/>
+</segment>
 </net>
